Commit message: Week 4: Complete - depth sensor skipped due to VMware limitation

File: urdf/robot.urdf.xacro (robot description, xacro)
@@ -1,10 +1,9 @@
 <?xml version="1.0"?>
 <!--
-robot.urdf.xacro – File gốc: gộp tất cả xacro lại thành 1 URDF
-================================================================
-robot_state_publisher đọc file này qua launch file.
-Thêm include mới ở đây khi cần mở rộng robot.
-Tuần 3: properties + materials + macros + robot_core
-Tuần 4: thêm gazebo_control + sensors (xem hướng dẫn bên dưới)
+  robot.urdf.xacro — File gốc: gộp tất cả xacro thành 1 URDF
+  =============================================================
+  TUẦN 4: thêm 2 include cho Gazebo simulation.
+  robot_state_publisher đọc file này qua launch file,
+  xử lý tất cả <xacro:include>, publish URDF lên /robot_description.
 -->
 <robot name="my_robot" xmlns:xacro="http://www.ros.org/wiki/xacro">
@@ -15,11 +14,9 @@
   <!-- Macro tính inertia -->
   <xacro:include filename="$(find my_robot_description)/urdf/macros.xacro"/>
-  <!-- Links + Joints của robot -->
+  <!-- Links + Joints (Tuần 3 + fixes Tuần 4) -->
   <xacro:include filename="$(find my_robot_description)/urdf/robot_core.xacro"/>
-  <!-- Sensors: camera + lidar -->
+  <!-- TUẦN 4 MỚI: DiffDrive plugin → robot nhận /cmd_vel, xuất /odom -->
+  <xacro:include filename="$(find my_robot_description)/urdf/gazebo_control.xacro"/>
+  <!-- TUẦN 4 MỚI: LiDAR → /scan, Camera → /camera/image_raw -->
   <xacro:include filename="$(find my_robot_description)/urdf/sensors.xacro"/>
-  <!--
-    TUẦN 4 – Thêm dòng này khi học Gazebo Simulation:
-    <xacro:include filename="$(find my_robot_description)/urdf/gazebo_control.xacro"/>
-  -->
 </robot>

File: urdf/robot_core.xacro (robot description, xacro)
@@ -3,22 +3,18 @@
   robot_core.xacro — Links & Joints của robot
   =============================================
-  Mô tả hình dạng vật lý: chassis, 2 drive wheels, 1 caster wheel.
-  File này chỉ chứa URDF thuần — không có Gazebo-specific tags.
-  Gazebo tags sẽ được thêm ở Tuần 4 (gazebo_control.xacro).
+  TUẦN 4 — 3 thay đổi so với Tuần 3:
+    1. Thêm <limit effort velocity> cho drive joints (tránh giật)
+    2. Drive wheels collision → sphere (giảm lateral friction)
+    3. Thêm <gazebo reference> caster → tắt ma sát
 -->
 <robot xmlns:xacro="http://www.ros.org/wiki/xacro">
-  <!-- ══════════════════════════════════════════════════
-       BASE FOOTPRINT — gốc tọa độ ảo trên mặt sàn
-       ══════════════════════════════════════════════════ -->
+  <!-- BASE FOOTPRINT -->
   <link name="base_footprint"/>
   <joint name="base_footprint_joint" type="fixed">
     <parent link="base_footprint"/>
     <child  link="base_link"/>
-    <!-- Nâng base_link lên đúng 1 wheel_radius so với sàn -->
     <origin xyz="0 0 ${wheel_radius}" rpy="0 0 0"/>
   </joint>
-  <!-- ══════════════════════════════════════════════════
-       BASE_LINK / CHASSIS — thân chính robot
-       ══════════════════════════════════════════════════ -->
+  <!-- CHASSIS -->
   <link name="base_link">
     <visual>
@@ -35,13 +31,10 @@
       </geometry>
     </collision>
-    <xacro:inertial_box
-      mass="${chassis_mass}"
+    <xacro:inertial_box mass="${chassis_mass}"
       x="${chassis_length}" y="${chassis_width}" z="${chassis_height}">
       <origin xyz="0 0 0" rpy="0 0 0"/>
     </xacro:inertial_box>
   </link>
-  <!-- ══════════════════════════════════════════════════
-       LEFT DRIVE WHEEL
-       ══════════════════════════════════════════════════ -->
+  <!-- LEFT DRIVE WHEEL -->
   <joint name="left_wheel_joint" type="continuous">
     <parent link="base_link"/>
@@ -49,4 +42,6 @@
     <origin xyz="0 ${wheel_ygap} ${wheel_zoff}" rpy="-${PI/2} 0 0"/>
     <axis xyz="0 0 1"/>
+    <!-- TUẦN 4: giới hạn lực (N.m) và tốc độ góc (rad/s) -->
+    <limit effort="0.05" velocity="10.0"/>
   </joint>
   <link name="left_wheel_link">
@@ -61,18 +56,14 @@
       <origin xyz="0 0 0" rpy="0 0 0"/>
       <geometry>
-        <!-- Sphere collision → giảm lateral friction (xem Tuần 4) -->
+        <!-- TUẦN 4: sphere → 1 điểm tiếp xúc, giảm lateral friction -->
         <sphere radius="${wheel_radius}"/>
       </geometry>
     </collision>
-    <xacro:inertial_cylinder
-      mass="${wheel_mass}"
-      radius="${wheel_radius}"
-      length="${wheel_width}">
+    <xacro:inertial_cylinder mass="${wheel_mass}"
+      radius="${wheel_radius}" length="${wheel_width}">
       <origin xyz="0 0 0" rpy="0 0 0"/>
     </xacro:inertial_cylinder>
   </link>
-  <!-- ══════════════════════════════════════════════════
-       RIGHT DRIVE WHEEL
-       ══════════════════════════════════════════════════ -->
+  <!-- RIGHT DRIVE WHEEL -->
   <joint name="right_wheel_joint" type="continuous">
     <parent link="base_link"/>
@@ -80,4 +71,6 @@
     <origin xyz="0 -${wheel_ygap} ${wheel_zoff}" rpy="${PI/2} 0 0"/>
     <axis xyz="0 0 1"/>
+    <!-- TUẦN 4: giới hạn lực và tốc độ -->
+    <limit effort="0.05" velocity="10.0"/>
   </joint>
   <link name="right_wheel_link">
@@ -92,22 +85,17 @@
       <origin xyz="0 0 0" rpy="0 0 0"/>
       <geometry>
+        <!-- TUẦN 4: sphere thay cylinder -->
         <sphere radius="${wheel_radius}"/>
       </geometry>
     </collision>
-    <xacro:inertial_cylinder
-      mass="${wheel_mass}"
-      radius="${wheel_radius}"
-      length="${wheel_width}">
+    <xacro:inertial_cylinder mass="${wheel_mass}"
+      radius="${wheel_radius}" length="${wheel_width}">
       <origin xyz="0 0 0" rpy="0 0 0"/>
     </xacro:inertial_cylinder>
   </link>
-  <!-- ══════════════════════════════════════════════════
-       CASTER WHEEL — bánh cân bằng phía sau
-       Fixed joint → không quay độc lập
-       ══════════════════════════════════════════════════ -->
+  <!-- CASTER WHEEL -->
   <joint name="caster_wheel_joint" type="fixed">
     <parent link="base_link"/>
     <child  link="caster_wheel_link"/>
-    <!-- Đặt phía sau, thấp hơn để chạm sàn -->
     <origin xyz="${caster_xoff} 0 ${wheel_zoff}" rpy="0 0 0"/>
   </joint>
@@ -126,9 +114,14 @@
       </geometry>
     </collision>
-    <xacro:inertial_sphere
-      mass="${caster_mass}"
-      radius="${caster_radius}">
+    <xacro:inertial_sphere mass="${caster_mass}" radius="${caster_radius}">
       <origin xyz="0 0 0" rpy="0 0 0"/>
     </xacro:inertial_sphere>
   </link>
+  <!-- TUẦN 4: tắt ma sát caster wheel
+       mu1/mu2 = 0 → caster quay tự do, không kéo robot khi quay,
+       odometry chính xác hơn -->
+  <gazebo reference="caster_wheel_link">
+    <mu1>0.0</mu1>
+    <mu2>0.0</mu2>
+  </gazebo>
 </robot>

File: urdf/sensors.xacro (robot description, xacro)
@@ -1,34 +1,131 @@
 <?xml version="1.0"?>
 <robot xmlns:xacro="http://www.ros.org/wiki/xacro">
-  <!-- CAMERA -->
-  <link name="camera_link">
+  <!-- LIDAR -->
+  <joint name="lidar_joint" type="fixed">
+    <parent link="base_link"/>
+    <child link="lidar_link"/>
+    <origin xyz="0 0 0.18" rpy="0 0 0"/>
+  </joint>
+  <link name="lidar_link">
     <visual>
-      <geometry><box size="0.03 0.05 0.03"/></geometry>
+      <geometry>
+        <cylinder length="0.04" radius="0.04"/>
+      </geometry>
       <material name="black"/>
     </visual>
+    <collision>
+      <geometry>
+        <cylinder length="0.04" radius="0.04"/>
+      </geometry>
+    </collision>
+    <inertial>
+      <mass value="0.1"/>
+      <inertia ixx="0.001" ixy="0" ixz="0"
+               iyy="0.001" iyz="0" izz="0.001"/>
+    </inertial>
   </link>
+  <gazebo reference="lidar_link">
+    <sensor type="ray" name="lidar_sensor">
+      <pose>0 0 0 0 0 0</pose>
+      <visualize>false</visualize>
+      <update_rate>10</update_rate>
+      <ray>
+        <scan>
+          <horizontal>
+            <samples>360</samples>
+            <resolution>1</resolution>
+            <min_angle>-3.14159</min_angle>
+            <max_angle>3.14159</max_angle>
+          </horizontal>
+        </scan>
+        <range>
+          <min>0.12</min>
+          <max>12.0</max>
+          <resolution>0.01</resolution>
+        </range>
+      </ray>
+      <plugin name="gazebo_ros_lidar"
+              filename="libgazebo_ros_ray_sensor.so">
+        <ros>
+          <remapping>~/out:=/scan</remapping>
+        </ros>
+        <frameName>lidar_link</frameName>
+      </plugin>
+    </sensor>
+  </gazebo>
+  <!-- CAMERA -->
   <joint name="camera_joint" type="fixed">
     <parent link="base_link"/>
     <child link="camera_link"/>
-    <origin xyz="0.15 0 0.05" rpy="0 0 0"/>
+    <origin xyz="0.155 0 0.05" rpy="0 0 0"/>
   </joint>
-  <!-- CAMERA OPTICAL -->
-  <link name="camera_optical_link"/>
+  <link name="camera_link">
+    <visual>
+      <geometry>
+        <box size="0.01 0.04 0.03"/>
+      </geometry>
+      <material name="red"/>
+    </visual>
+    <inertial>
+      <mass value="0.05"/>
+      <inertia ixx="0.0001" ixy="0" ixz="0"
+               iyy="0.0001" iyz="0" izz="0.0001"/>
+    </inertial>
+  </link>
   <joint name="camera_optical_joint" type="fixed">
     <parent link="camera_link"/>
     <child link="camera_optical_link"/>
-    <origin xyz="0 0 0" rpy="${-pi/2} 0 ${-pi/2}"/>
+    <origin xyz="0 0 0" rpy="-1.5707963 0 -1.5707963"/>
   </joint>
-  <!-- LIDAR -->
-  <link name="lidar_link">
-    <visual>
-      <geometry><cylinder radius="0.04" length="0.05"/></geometry>
-      <material name="black"/>
-    </visual>
-  </link>
-  <joint name="lidar_joint" type="fixed">
-    <parent link="base_link"/>
-    <child link="lidar_link"/>
-    <origin xyz="0 0 0.08" rpy="0 0 0"/>
-  </joint>
+  <link name="camera_optical_link"/>
+  <gazebo reference="camera_link">
+    <sensor type="camera" name="camera_sensor">
+      <update_rate>30</update_rate>
+      <camera name="head">
+        <horizontal_fov>1.3962634</horizontal_fov>
+        <image>
+          <width>640</width>
+          <height>480</height>
+          <format>R8G8B8</format>
+        </image>
+        <clip>
+          <near>0.02</near>
+          <far>300</far>
+        </clip>
+      </camera>
+      <plugin name="gazebo_ros_camera"
+              filename="libgazebo_ros_camera.so">
+        <cameraName>camera</cameraName>
+        <imageTopicName>/camera/image_raw</imageTopicName>
+        <cameraInfoTopicName>/camera/camera_info</cameraInfoTopicName>
+        <frameName>camera_link</frameName>
+      </plugin>
+    </sensor>
+  </gazebo>
+  <!-- DEPTH CAMERA -->
+  <gazebo reference="camera_link">
+    <sensor type="depth" name="depth_sensor">
+      <update_rate>30</update_rate>
+      <camera name="depth">
+        <horizontal_fov>1.3962634</horizontal_fov>
+        <image>
+          <width>640</width>
+          <height>480</height>
+          <format>R8G8B8</format>
+        </image>
+        <clip>
+          <near>0.02</near>
+          <far>300</far>
+        </clip>
+      </camera>
+      <plugin name="gazebo_ros_depth_camera"
+          filename="libgazebo_ros_camera.so">
+    <ros>
+      <remapping>~/image_raw:=/depth/image_raw</remapping>
+      <remapping>~/depth/image_raw:=/depth/image_raw</remapping>
+    </ros>
+    <frameName>camera_link</frameName>
+     </plugin>
+    </sensor>
+  </gazebo>
 </robot>
